File: elec/alim/alim.kicad_pcb (KiCad board)
At the start: 2 copper layers, 58.4 x 108 mm, 30 parts, among them J11 Conn_01x02_Male, J12 Conn_01x02_Male, J21 Conn_01x02_Male, J22 Conn_01x02_Male, J23 Conn_01x02_Male, J3 Conn_01x02_Male, J4 Conn_01x02_Male, J51 Conn_01x02_Male, J52 Conn_01x02_Male, K3 G5LE-1, U1 LM2576T-5, U2 LM2576T-5

Commit message: debut uniformisation des trous
Connections:
- K3 pad 3: Net-(K3-Pad3) -> /Vpow
- K3 pad 4: /Vpow -> Net-(K3-Pad4)
Routing:
- net /Vpow: track 15.6 -> 28.3 mm
- net GND: track 252.9 -> 262.8 mm
