File: elec/alim/alim.kicad_pcb (KiCad board)
At the start: 2 copper layers, 58.4 x 108 mm, 30 parts, among them J11 Conn_01x02_Male, J12 Conn_01x02_Male, J21 Conn_01x02_Male, J22 Conn_01x02_Male, J23 Conn_01x02_Male, J3 Conn_01x02_Male, J4 Conn_01x02_Male, J51 Conn_01x02_Male, J52 Conn_01x02_Male, K3 G5LE-1, U1 LM2576T-5, U2 LM2576T-5

Commit message: modif fusibles
Parts:
- F1, F2, F5: footprint Fuse:Fuse_Blade_ATO_directSolder -> fuse:fusible_alim
- J23: footprint Connector_Wire:SolderWire-1sqmm_1x02_P5.4mm_D1.4mm_OD2.7mm -> Connector_Wire:SolderWire-0.127sqmm_1x02_P3.7mm_D0.48mm_OD1mm
- moved F1 16.5 mm to (114.3, 6.85), turned to 270 degrees
- moved F2 12.3 mm to (105.6, 10.2), turned to 90 degrees
- moved F5 11.7 mm to (105.6, 0.15), turned to 90 degrees
- moved C21 7.18 mm to (96.5, 21.6)
- moved L2 5.08 mm to (83.8, 29.2)
- moved U2 4.58 mm to (100.3, 29.2)
- moved U1 3.81 mm to (133.3, 26.7)
- moved J23 3.59 mm to (86.4, 62.2), turned to 0 degrees
- moved C11 2.84 mm to (129.5, 17.8)
- moved L1 2.54 mm to (116.8, 29.2)
- moved J4 2.29 mm to (131.4, -14.0)
Routing:
- net /Vpow: track 28.3 -> 54.4 mm
- net /Vbat: track 45.6 -> 35.2 mm
- net GND: track 262.8 -> 268.3 mm
- net Net-(C21-Pad1): track 24.5 -> 29.0 mm
- net Net-(F5-Pad1): track 28.2 -> 24.4 mm
- net Net-(C12-Pad1): track 51.5 -> 55.3 mm
- net Net-(C11-Pad1): track 23.0 -> 26.5 mm
- net Net-(L2-Pad1): track 15.3 -> 18.3 mm
- net Net-(L1-Pad1): track 14.0 -> 15.6 mm
Other:
- board text added: "alert"
- board text removed: "+ G"
- board text removed: "sense"

Commit message: modif finales et impression
Parts:
- added D4: LED, LED_THT:LED_D3.0mm, F.Cu at (118.1, -27.9)
- added G***: LOGO, logo:logo, F.Cu at (114.9, 66.0)
- added R4: R, Resistor_THT:R_Axial_DIN0411_L9.9mm_D3.6mm_P12.70mm_Horizontal, F.Cu at (125.7, -15.2)
- moved J4 2.84 mm to (134.0, -15.2)
- moved J12 2.54 mm to (127.0, 74.9)
- moved J22 2.54 mm to (101.6, 74.9)
- moved REF** 2.54 mm to (86.4, 74.9)
- moved REF** 2.54 mm to (134.6, 74.9)
- moved J51 2.54 mm to (90.2, -21.6)
- moved REF** 2.54 mm to (86.4, -29.2)
- moved REF** 2.54 mm to (134.6, -29.2)
- moved J11 0.64 mm to (127.0, 62.9)
- moved J21 0.64 mm to (101.6, 62.9)
Routing:
- net /Vbat: track 35.2 -> 56.4 mm
- net GND: track 268.3 -> 262.7 mm
- net Net-(D4-Pad2): track 0.00 -> 5.08 mm
- net Net-(C12-Pad1): track 55.3 -> 58.5 mm
- net Net-(F5-Pad1): track 24.4 -> 27.0 mm
- net Net-(C22-Pad1): track 60.0 -> 62.6 mm
Other:
- board size 58.4 x 108 mm -> 58.4 x 113 mm
- board text added: "Comment appelle-t-on un boomerang qui ne revient pas ?"
- board text added: "un bout de bois !"
