File: elec/alim/alim.sch (KiCad schematic (older format))
At the start: 26 parts, among them J11 Conn_01x02_Male, J12 Conn_01x02_Male, J21 Conn_01x02_Male, J22 Conn_01x02_Male, J23 Conn_01x02_Male, J3 Conn_01x02_Male, J4 Conn_01x02_Male, J51 Conn_01x02_Male, J52 Conn_01x02_Male, K3 G5LE-1, U1 LM2576T-5, U2 LM2576T-5

Commit message: debut uniformisation des trous
Connections:
- net Vpow: now also K3.3; no longer K3.4
Changed lines of the file:
@@
 Wire Wire Line
 	1900 4950 1900 4650
-Text Label 1800 3850 0    50   ~ 0
+Text Label 2000 3950 0    50   ~ 0
 Vpow
-Wire Wire Line
-	1800 3850 1800 4050
 $Comp
 L Device:Fuse F2
@@
 Wire Wire Line
 	9800 3750 9000 3750
-NoConn ~ 2000 4050
+NoConn ~ 1800 4050
 $Comp
 L Device:Fuse F5
@@
 Wire Wire Line
 	9700 5200 9000 5200
+Wire Wire Line
+	2000 3950 2000 4050
 $EndSCHEMATC

Commit message: modif fusibles
Parts:
- F1, F2, F5: footprint Fuse:Fuse_Blade_ATO_directSolder -> fuse:fusible_alim
- J23: footprint Connector_Wire:SolderWire-1sqmm_1x02_P5.4mm_D1.4mm_OD2.7mm -> Connector_Wire:SolderWire-0.127sqmm_1x02_P3.7mm_D0.48mm_OD1mm
Changed lines of the file:
@@
 F 0 "F1" V 3953 3550 50  0000 C CNN
 F 1 "5A" V 4044 3550 50  0000 C CNN
-F 2 "Fuse:Fuse_Blade_ATO_directSolder" V 4080 3550 50  0001 C CNN
+F 2 "fuse:fusible_alim" V 4080 3550 50  0001 C CNN
 F 3 "~" H 4150 3550 50  0001 C CNN
 	1    4150 3550
@@
 F 0 "F2" V 3953 5000 50  0000 C CNN
 F 1 "5A" V 4044 5000 50  0000 C CNN
-F 2 "Fuse:Fuse_Blade_ATO_directSolder" V 4080 5000 50  0001 C CNN
+F 2 "fuse:fusible_alim" V 4080 5000 50  0001 C CNN
 F 3 "~" H 4150 5000 50  0001 C CNN
 	1    4150 5000
@@
 F 0 "J23" H 10622 5532 50  0000 R CNN
 F 1 "Conn_01x02_Male" H 10622 5623 50  0000 R CNN
-F 2 "Connector_Wire:SolderWire-1sqmm_1x02_P5.4mm_D1.4mm_OD2.7mm" H 10650 5650 50  0001 C CNN
+F 2 "Connector_Wire:SolderWire-0.127sqmm_1x02_P3.7mm_D0.48mm_OD1mm" H 10650 5650 50  0001 C CNN
 F 3 "~" H 10650 5650 50  0001 C CNN
 	1    10650 5650
@@
 F 0 "F5" V 7003 1600 50  0000 C CNN
 F 1 "10A" V 7094 1600 50  0000 C CNN
-F 2 "Fuse:Fuse_Blade_ATO_directSolder" V 7130 1600 50  0001 C CNN
+F 2 "fuse:fusible_alim" V 7130 1600 50  0001 C CNN
 F 3 "~" H 7200 1600 50  0001 C CNN
 	1    7200 1600

Commit message: modif finales et impression
Parts:
- added D4: LED, LED_THT:LED_D3.0mm, symbol Device:LED
- added R4: R, Resistor_THT:R_Axial_DIN0411_L9.9mm_D3.6mm_P5.08mm_Vertical, symbol Device:R
Connections:
- net GND: now also D4.1 (K)
- net Vbat: now also R4.1
- new net: D4.2 (A), R4.2
Changed lines of the file:
@@
 Wire Wire Line
 	2000 3950 2000 4050
+$Comp
+L Device:LED D4
+U 1 1 603904F4
+P 2450 1600
+F 0 "D4" V 2489 1482 50  0000 R CNN
+F 1 "LED" V 2398 1482 50  0000 R CNN
+F 2 "LED_THT:LED_D3.0mm" H 2450 1600 50  0001 C CNN
+F 3 "~" H 2450 1600 50  0001 C CNN
+	1    2450 1600
+	0    -1   -1   0
+$EndComp
+Text Label 2450 1100 0    50   ~ 0
+Vbat
+$Comp
+L Device:R R4
+U 1 1 60391A95
+P 2450 1250
+F 0 "R4" H 2520 1296 50  0000 L CNN
+F 1 "R" H 2520 1205 50  0000 L CNN
+F 2 "Resistor_THT:R_Axial_DIN0411_L9.9mm_D3.6mm_P5.08mm_Vertical" V 2380 1250 50  0001 C CNN
+F 3 "~" H 2450 1250 50  0001 C CNN
+	1    2450 1250
+	1    0    0    -1
+$EndComp
+Wire Wire Line
+	2450 1450 2450 1400
+$Comp
+L power:GND #PWR0107
+U 1 1 60394F80
+P 2450 1750
+F 0 "#PWR0107" H 2450 1500 50  0001 C CNN
+F 1 "GND" H 2455 1577 50  0000 C CNN
+F 2 "" H 2450 1750 50  0001 C CNN
+F 3 "" H 2450 1750 50  0001 C CNN
+	1    2450 1750
+	1    0    0    -1
+$EndComp
 $EndSCHEMATC
